File: MicroDV_PCB_Schematics/MicroDV2/MicroDV2.kicad_sch (KiCad schematic)
At the start: 79 parts, among them J10 Conn_02x03, J6 Conn_02x18_Counter_Clockwise, J7 Conn_01x02, J8 Conn_01x02, J9 Conn_01x02, K1 3-1393237-1, K2 Relay_DPDT, Q1 AOD4185, Q3 AO3434A, Q4 AO3434A, Q5 AO3434A, Q6 BCV29, Q7 BCV29, Q8 AOD4185, SW1 SW_DIP_x01, U2 OKI-78SR-12_1.0-W36H-C, U3 OKI-78SR-5_1.5-W36-C

Commit message: MicroDV pre feedback
Parts:
- removed R23: 1k, ISC_paquetes:0805_PAN, symbol Device:R
- removed R25: 10k, ISC_paquetes:0805_PAN, symbol Device:R
Connections:
- net ASSI blue in (-): now also DZ2.1 (K), Q8.2 (S), R36.1; no longer Q8.3 (D), R38.1
- net ASSI blue out (+): no longer DZ1.1 (K), DZ2.1 (K), Q1.2 (S), Q8.2 (S), R2.1, R36.1
- net ASSI yellow in (-): now also DZ1.1 (K), Q1.2 (S), R2.1; no longer Q1.3 (D), R1.1
- new net: Q1.3 (D), R1.1
- new net: Q8.3 (D), R38.1
