File: MicroDV_PCB_Schematics/MicroDV2/MicroDV2.kicad_sch (KiCad schematic)
At the start: 87 parts, among them J10 Conn_02x03, J6 Conn_02x18_Counter_Clockwise, J7 Conn_01x02, J8 Conn_01x02, J9 Conn_01x02, K1 RT425012, K3 RT33L024, Q1 AOD4185, Q10 BC856B, Q11 PMV37ENEA, Q2 PMV37ENEA, Q3 BC846B, Q4 BC856B, Q5 AO3434A, Q6 BCV29, Q7 BCV29, Q8 AOD4185, Q9 BC846B, SW1 SW_DIP_x01, U2 OKI-78SR-12_1.0-W36H-C, U3 OKI-78SR-5_1.5-W36-C

Commit message: Filtros paso bajo
Parts:
- added C5, C6: 1u, Capacitor_SMD:C_0805_2012Metric, symbol Device:C
- added C7, C8: 270n, Capacitor_SMD:C_0805_2012Metric, symbol Device:C
Connections:
- net 24V is gone; now on net 24V de LVMS GF: SW1.2
- net ASMS 2 (24V) is gone; now on net 24V EBS: D1.1 (K), D2.1 (K), J10.1 (+12V), J10.4 (GND), J10.5 (GND), K3.11, Q10.3 (C), Q4.3 (C), R23.1, R42.1, R43.1, R5.1
- net ASMS gnd Steering Motor is gone; now on net GND: J10.3 (GND)
- net GND: now also C5.2, C6.2, C7.2, C8.2
- net Lectura RES (A5): now also C6.1
- net Micro in EBS (A3): now also C5.1
- net Micro in pres 1 (A1): now also C7.1
- net Micro in pres 2 (A2): now also C8.1
Other:
- note added: "PARA TESTEAR FUERA DEL VEHICULO (desoldar al meter en el coche)"
- note added: "fc=175 Hz (paso bajo)"
- moved on the sheet: R40, R41
