File: MicroDV_PCB_Schematics/MicroDV2/_restore_backup_2026-10-05T11-19-40-120/MicroDV2.kicad_sch (KiCad schematic)
At the start: 87 parts, among them J10 Conn_02x03, J6 Conn_02x18_Counter_Clockwise, J7 Conn_01x02, J8 Conn_01x02, J9 Conn_01x02, K1 RT425012, K3 RT33L024, Q1 AOD4185, Q10 BC856B, Q11 PMV37ENEA, Q2 PMV37ENEA, Q3 BC846B, Q4 BC856B, Q5 AO3434A, Q6 BCV29, Q7 BCV29, Q8 AOD4185, Q9 BC846B, SW1 SW_DIP_x01, U2 OKI-78SR-12_1.0-W36H-C, U3 OKI-78SR-5_1.5-W36-C

Commit message: Feedback aplicado
Parts:
- removed K3: RT33L024, Relay_THT:Relay_SPST_Schrack-RT1-16A-FormA_RM5mm, symbol Relay:FINDER-32.21-x300
- added D10, D11: LED, ISC_electromecanica:150080RS75000_WRE, symbol Device:LED
- added K2: Relay_DPDT, ISC_paquetes:RTE24012, symbol Relay:Relay_DPDT
- added R24: 1k, ISC_paquetes:0805_PAN, symbol Device:R
- added R39: 120, ISC_paquetes:0805_PAN, symbol Device:R
- K1: value RT425012 -> 3-1393237-1; footprint Relay_THT:Relay_DPDT_Schrack-RT2-FormC_RM5mm -> ISC_conectores:TE_3-1393237-1
Connections:
- net 12V de LVMS: now also D10.2 (A), D11.2 (A)
- net ASMS 2 (24V): now also K2.11
- net ASMS in 1: now also K2.14
- net CAN H 2: now also R39.2
- net CAN L 2: now also R39.1
- net Control SDC: now also Q5.2 (D); no longer Q5.3 (S)
- net GND: now also Q5.3 (S), R24.1; no longer D19.2 (A), Q5.2 (D)
- net SDC out renamed SDC 2
- net SDC 2: now also D19.2 (A), K2.A2; no longer D19.1 (K), J7.2 (Pin_2)
- new net: K2.21, R24.2
- new net: D11.1 (K), K2.22
- new net: D10.1 (K), K2.24
- new net SDC 3 out: D19.1 (K), J7.2 (Pin_2), K2.A1
- no-connect marks 14 -> 15
Other:
- note added: "El relé de la libreria es de 24V, aquí necesito uno de 12V. Por eso no es de la libreria. Lo he cogido del anterior diseño de la placa de steering"
- note added: "Estos modelos de regulador lineal los he sacado de la anterior placa de steering, del rediseño de Andrés"
